File: OBJEX-DoorSensor_v1.2/OBJEX-DoorSensor_v1.2.kicad_pcb (KiCad board)
At the start: 2 copper layers, 65 parts, among them Q1 BC857B_RF, Q2 NTNUS3171PZT5G, Q3 2N7002KQBZ, Q4 BSS138, Q5 BSS138, Q6 DMG3415UFY4Q-7, U2 RT9080-33GJ5, U3 S-5701BC11B-L3T2U5, U4 SN74LVC1G86DBVR, U5 SN74LVC1G86DBVR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

Commit message: update
Parts:
- moved C8 4.41 mm to (91.0, 76.5)
- moved C9 4.41 mm to (91.0, 79.0)
- moved Q1 4.41 mm to (107.6, 77.5)
- moved R5 4.41 mm to (91.0, 84.0)
- moved C10 4.41 mm to (91.0, 81.5)
- moved C11 4.41 mm to (106.1, 85.3)
- moved C12 4.41 mm to (106.1, 87.3)
- moved Q2 4.41 mm to (106.2, 89.2)
- moved Q6 4.41 mm to (106.5, 81.9)
- moved R6 4.41 mm to (91.0, 86.5)
- moved R7 4.41 mm to (91.0, 89.1)
- moved Q3 4.41 mm to (110.4, 82.0)
- moved R10 4.41 mm to (94.4, 80.2)
- moved R12 4.41 mm to (94.4, 84.2)
- moved R13 4.41 mm to (94.4, 86.2)
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
Commit message: update
Parts:
- moved U4 30.1 mm to (72.6, 77.0)
- moved C12 27.1 mm to (80.6, 78.2), turned to -90 degrees
- moved R6 24.9 mm to (71.8, 70.7), turned to -90 degrees
- moved Q2 24.8 mm to (87.2, 73.3), turned to 90 degrees
- moved R7 24.4 mm to (71.8, 74.0), turned to -90 degrees
- moved R5 23.8 mm to (69.4, 74.0), turned to -90 degrees
- moved U5 20.9 mm to (83.1, 77.8)
- moved Q1 20.8 mm to (86.8, 77.4), turned to 90 degrees
- moved Q3 20.1 mm to (90.3, 80.4)
- moved R9 19.9 mm to (74.6, 79.9), turned to 180 degrees
- moved R8 19.5 mm to (75.0, 78.2), turned to -90 degrees
- moved Q6 19.0 mm to (89.6, 73.3)
- moved R10 17.8 mm to (76.8, 77.7)
- moved R14 12.9 mm to (97.6, 75.7)
- moved R13 12.9 mm to (97.6, 73.7)
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
Commit message: update
Parts:
- removed D4: SP0503BAHT, Package_TO_SOT_SMD:SOT-143
- added D5: 1N4148WS, Diode_SMD:D_SOD-323, F.Cu at (139.2, 118.8)
- added G***: LOGO, libMaster:Xlogo, F.Cu at (153.5, 77.0)
- added G***: LOGO, KicadLibrary:logov2-mini, F.Cu at (152.2, 121.0)
- added JP1: SolderJumper_2_Open, Jumper:SolderJumper-2_P1.3mm_Open_RoundedPad1.0x1.5mm, F.Cu at (136.8, 118.8)
- added kibuzzard-63AF0800: G***, kibuzzard-63AF0800, F.Cu at (137.1, 128.6)
- added kibuzzard-63AF0810: G***, kibuzzard-63AF0810, F.Cu at (152.5, 128.8)
- C10, C9: footprint Capacitor_SMD:C_0603_1608Metric -> Capacitor_SMD:C_0402_1005Metric
- TP1, TP2: moved to B.Cu
- moved R6 91.5 mm to (151.2, 116.0), turned to 0 degrees
- moved R5 90.5 mm to (151.2, 112.5), turned to 0 degrees
- moved R7 89.1 mm to (151.2, 114.2), turned to 0 degrees
- moved U4 83.6 mm to (148.0, 113.0), turned to 180 degrees
- moved R9 80.1 mm to (148.5, 110.7), turned to -90 degrees
- moved R8 79.2 mm to (147.2, 110.7), turned to 90 degrees
- moved R10 76.7 mm to (146.0, 110.8), turned to 90 degrees
- moved C8 71.0 mm to (142.0, 111.0), turned to 90 degrees
- moved C12 71.0 mm to (144.0, 110.0), turned to 90 degrees
- moved U5 70.2 mm to (144.0, 112.6), turned to -90 degrees
- moved R11 65.6 mm to (141.5, 107.2), turned to 180 degrees
- moved Q1 63.2 mm to (139.0, 113.0), turned to 180 degrees
- moved Q2 62.1 mm to (140.2, 105.5)
- moved Q6 58.3 mm to (138.2, 105.3)
- moved R13 57.0 mm to (143.2, 107.8), turned to -90 degrees
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Connections:
- TP1 pad 1: +BATT -> Net-(D5-A)
Other:
- board outline added: 20 x 50.2 mm

Commit message: Start PCB design
Parts:
- removed kibuzzard-63AF0810: G***, kibuzzard-63AF0810
- added G***: LOGO, KicadLibrary:logov2-mini, B.Cu at (145.0, 112.2)
- added U1: 5204, BatteryTerminal:5204, F.Cu at (150.8, 118.5)
- added U10: 5226, BatteryTerminal:5226, F.Cu at (139.3, 112.0)
- added kibuzzard-64258E17: G***, kibuzzard-64258E17, F.Cu at (150.8, 115.6)
- added kibuzzard-64258E23: G***, kibuzzard-64258E23, F.Cu at (139.2, 115.4)
- added kibuzzard-64258E45: G***, kibuzzard-64258E45, F.Cu at (152.0, 124.4)
- added kibuzzard-64258E65: G***, kibuzzard-64258E65, F.Cu at (136.4, 101.2)
- added kibuzzard-64258FE0: G***, kibuzzard-64258FE0, B.Cu at (150.8, 120.4)
- kibuzzard-63AF0800: moved to B.Cu
- moved G*** 45.2 mm to (152.2, 122.2)
- moved G*** 40.2 mm to (153.4, 80.8)
- moved kibuzzard-63AF0800 8.42 mm to (139.2, 120.4), turned to 180 degrees
- moved D5 3.70 mm to (139.4, 122.5), turned to 90 degrees
- moved JP1 3.65 mm to (136.8, 122.4), turned to -90 degrees
- moved R20 1.88 mm to (141.8, 115.0), turned to 180 degrees
- moved R3 1.88 mm to (148.2, 115.0), turned to 0 degrees
- moved R5 1.71 mm to (151.4, 110.8)
- moved R6 1.71 mm to (151.4, 114.3)
- moved R7 1.71 mm to (151.4, 112.5)
- moved TP1 1.70 mm to (139.2, 122.6)
- moved U3 1.60 mm to (146.8, 98.4)
- moved S1 1.60 mm to (152.6, 98.4)
- moved C8 1.55 mm to (142.4, 109.5)
- moved TP2 1.50 mm to (150.8, 122.6)
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Routing:
- net /Microcontroller + WiFi-BLE/EN: track 0.00 -> 62.2 mm, vias 0 -> 3
- net +BATT: track 0.00 -> 52.3 mm, vias 0 -> 2
- net /Microcontroller + WiFi-BLE/LED_BLUE: track 0.00 -> 36.5 mm, vias 0 -> 2
- net /Microcontroller + WiFi-BLE/LED_GREEN: track 0.00 -> 36.0 mm, vias 0 -> 2
- net /Microcontroller + WiFi-BLE/LED_RED: track 0.00 -> 34.7 mm, vias 0 -> 2
- net /Microcontroller + WiFi-BLE/AUTO_TURN_OFF: track 0.00 -> 31.7 mm, vias 0 -> 2
- net Net-(U3-OUT): track 0.00 -> 27.5 mm, vias 0 -> 2
- net +3V3: track 0.00 -> 18.2 mm
- net Net-(JP3-A): track 0.00 -> 14.1 mm
- net /Power Latch - Rising & falling edge detector /Gate: track 0.00 -> 12.1 mm
- net Net-(D5-A): track 0.00 -> 8.92 mm, vias 0 -> 1
- net Net-(U5A-B): track 0.00 -> 5.64 mm
- net Net-(U2-EN): track 0.00 -> 4.57 mm
- net /Microcontroller + WiFi-BLE/GPIO0: track 0.00 -> 4.52 mm
- net /Microcontroller + WiFi-BLE/GPIO1: track 0.00 -> 4.52 mm
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- added copper zone on B.Cu, net GND
- added copper zone on F.Cu, net GND
- added copper zone on F.Cu, net VCC

Commit message: update
Parts:
- moved R17 5.59 mm to (142.5, 96.8), turned to 90 degrees
- moved R16 2.47 mm to (142.5, 94.0), turned to 90 degrees
- moved Q4 1.64 mm to (145.0, 90.7)
- moved Q5 1.00 mm to (140.0, 95.4)
- moved R18 0.25 mm to (147.8, 94.5)
- moved C14 0.20 mm to (145.7, 98.8)
- moved G*** 0.10 mm to (153.5, 80.8)
Routing:
- net +3V3: track 18.2 -> 55.2 mm, vias 0 -> 2
- net /Microcontroller + WiFi-BLE/BATT_LVL: track 2.93 -> 36.9 mm, vias 0 -> 2
- net /Microcontroller + WiFi-BLE/IN_STATUS: track 1.25 -> 27.1 mm, vias 0 -> 2
- net +1V8: track 0.00 -> 25.7 mm
- net /Microcontroller + WiFi-BLE/TX/GPIO21: track 0.00 -> 23.2 mm, vias 0 -> 2
- net /Microcontroller + WiFi-BLE/RX/GPIO20: track 0.00 -> 22.8 mm, vias 0 -> 2
- net /Microcontroller + WiFi-BLE/DTR/GPIO9: track 0.00 -> 21.9 mm, vias 0 -> 2
- net GND: track 0.00 -> 18.1 mm, vias 0 -> 17
- net /Microcontroller + WiFi-BLE/GPIO2: track 2.54 -> 16.9 mm, vias 0 -> 2
- net /Microcontroller + WiFi-BLE/GPIO8: track 0.00 -> 6.74 mm
- net Net-(Q5-S): track 0.00 -> 5.68 mm
- net Net-(JP3-A): track 14.1 -> 19.7 mm
- net Net-(Q4-S): track 0.00 -> 5.29 mm
- net /Microcontroller + WiFi-BLE/AUTO_TURN_OFF: track 31.7 -> 28.4 mm
- net Net-(U6-CSB): track 0.00 -> 2.80 mm
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- added copper zone on F.Cu, net +3V3

Commit message: Ready for last review
Parts:
- removed kibuzzard-64258E45: G***, kibuzzard-64258E45
- added kibuzzard-64258E17: G***, kibuzzard-64258E17, B.Cu at (150.8, 115.6)
- added kibuzzard-64258E23: G***, kibuzzard-64258E23, B.Cu at (139.2, 115.4)
- added kibuzzard-642BF081: G***, kibuzzard-642BF081, B.Cu at (144.9, 111.8)
- added kibuzzard-642BF0F2: G***, kibuzzard-642BF0F2, F.Cu at (150.8, 124.0)
- moved G*** 2.70 mm to (145.0, 109.5)
- moved G*** 1.57 mm to (150.8, 121.6)
Routing:
- net GND: track 18.1 -> 22.3 mm
Other:
- board text added: "0"
- board text added: "0 mm"
- board text added: "0.01 mm"
- board text added: "0.02"
- board text added: "0.035 mm"
- board text added: "0.2000 mm / 0.0000 mm"
- board text added: "0.3000 mm"
- board text added: "0.71 mm"
- board text added: "0.8000 mm"
- board text added: "1"
- board text added: "2"
- board text added: "20.0000 mm x 50.1893 mm"
- board text added: "3.3"
- board text added: "4.5"
- board text added: "ANT ZONE"
- board text added: "B.Cu"
- board text added: "B.Mask"
- board text added: "B.Paste"
- board text added: "B.Silkscreen"
- board text added: "BOARD CHARACTERISTICS"
- board text added: "Board Thickness:"
- board text added: "Board overall dimensions:"
- board text added: "Bottom Silk Screen"
- board text added: "Bottom Solder Mask"
- board text added: "Bottom Solder Paste"
- board text added: "Castellated pads:"
- board text added: "Color"
- board text added: "Copper Finish:"
- board text added: "Copper Layer Count:"
- board text added: "Dielectric 1"
- board text added: "Edge card connectors:"
- board text added: "Epsilon R"
- board text added: "F.Cu"
- board text added: "F.Mask"
- board text added: "F.Paste"
- board text added: "F.Silkscreen"
- board text added: "FR4"
- board text added: "Impedance Control:"
- board text added: "Layer Name"
- board text added: "Loss Tangent"
- board text added: "Material"
- board text added: "Min hole diameter:"
- board text added: "Min track/spacing:"
- board text added: "No"
- board text added: "None"
- board text added: "Not specified"
- board text added: "Plated Board Edge:"
- board text added: "Thickness (mm)"
- board text added: "Top Silk Screen"
- board text added: "Top Solder Mask"
- board text added: "Top Solder Paste"
- board text added: "Type"
- board text added: "copper"
- board text added: "core"
- board text added: "locked"

Commit message: last review
Parts:
- moved R10 0.60 mm to (145.9, 110.5), turned to 180 degrees
- moved C8 0.20 mm to (142.4, 109.7)
Routing:
- net Net-(U5A-B): track 5.60 -> 4.27 mm

Commit message: Ready for order
Parts:
- moved G*** 0.25 mm to (145.0, 109.8)
- moved kibuzzard-64258E23 0.15 mm to (139.2, 115.2) (x2)
Routing:
- net /Microcontroller + WiFi-BLE/LED_RED: track 36.7 -> 35.8 mm
- net /Microcontroller + WiFi-BLE/LED_GREEN: track 36.0 -> 35.1 mm
- net /Microcontroller + WiFi-BLE/LED_BLUE: track 37.9 -> 37.1 mm
- net GND: vias 17 -> 78
