File: OBJEX-DoorSensor_v1.2/OBJEX-DoorSensor_v1.2.kicad_pcb (KiCad board)
At the start: 2 copper layers, 20 x 50.2 mm, 80 parts, among them Q1 BC857B_RF, Q2 NTNUS3171PZT5G, Q3 2N7002KQBZ, Q4 BSS138, Q5 BSS138, Q6 DMG3415UFY4Q-7, U1 5204, U10 5226, U2 RT9080-33GJ5, U3 S-5701BC11B-L3T2U5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

Commit message: Final review - ready for production
Parts:
- added R22: 100K, Resistor_SMD:R_0402_1005Metric, F.Cu at (136.2, 109.5)
- added R23: 1K, Resistor_SMD:R_0402_1005Metric, F.Cu at (141.8, 113.4)
- R12: value 1K -> 10K
- moved R12 1.94 mm to (136.2, 107.2), turned to 90 degrees
Connections:
- Q1 pad 1: Net-(U5A-Y) -> Net-(Q1-Pad1)
- Q3 pad 1: /Microcontroller + WiFi-BLE/AUTO_TURN_OFF -> Net-(Q3-Pad1)
- Q3 pad 2: Net-(Q3-Pad2) -> GND
- R12 pad 1: Net-(Q3-Pad2) -> Net-(Q3-Pad1)
- R12 pad 2: GND -> /Microcontroller + WiFi-BLE/AUTO_TURN_OFF
Routing:
- net Net-(Q3-Pad1): track 0.00 -> 4.54 mm
- net /Microcontroller + WiFi-BLE/LED_GREEN: track 35.1 -> 39.6 mm
- net Net-(U5A-Y): track 3.98 -> 1.04 mm
- net /Microcontroller + WiFi-BLE/AUTO_TURN_OFF: track 28.4 -> 30.6 mm
- net Net-(Q3-Pad2): track 2.02 -> 0.00 mm
- net Net-(Q1-Pad1): track 0.00 -> 1.92 mm
- net GND: track 22.3 -> 24.1 mm, vias 78 -> 79
