File: OBJEX-DoorSensor_v1.2/BME680.kicad_sch (KiCad schematic)
At the start: 10 parts, among them Q4 BSS138, Q5 BSS138, U6 BME680, U8 MCP1802T-1802I/OT

Commit message: SCH complate
Other:
- company: (none) -> OBJEX
- title: (none) -> DW Sensor Module - (No modular design)

Commit message: update
Other:
- note added: "Copyright CERN 2020. This source describes Open Hardware and is licensed under the CERN-OHLW v2 You may redistribute and modify this documentation and make products using it under the terms of the CERN-OHL-W v2 (https:/cern.ch/cern-ohl). This documentation is distributed WITHOUT ANY EXPRESS OR IMPLIED WARRANTY, INCLUDING OF MERCHANTABILITY, SATISFACTORY QUALITY AND FITNESS FOR A PARTICULAR PURPOS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"
Changed lines of the file:
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@@
     (effects (font (size 4 4) (thickness 0.6) bold) (justify left bottom))
+  )
+  (text "Copyright CERN 2020.\nThis source describes Open Hardware and is licensed under the CERN-OHLW v2\nYou may redistribute and modify this documentation and make products\nusing it under the terms of the CERN-OHL-W v2 (https:/cern.ch/cern-ohl).\nThis documentation is distributed WITHOUT ANY EXPRESS OR IMPLIED\nWARRANTY, INCLUDING OF MERCHANTABILITY, SATISFACTORY QUALITY\nAND FITNESS FOR A PARTICULAR PURPOSE. Please see the CERN-OHL-W v2\nfor applicable conditions.\nSource location: https://www.ohwr.org/project/wr-switch-hw\nAs per CERN-OHL-W v2 section 4.1, should You produce hardware based on\nthese sources, You must maintain the Source Location visible on the\nexternal case of the White Rabbit switch or other product you make using\nthis documentation."
+    (at 16.51 195.58 0)
+    (effects (font (size 2 2)) (justify left bottom))
   )
   (hierarchical_label "SDA" (shape bidirectional) (at 248.3358 97.155 0) (fields_autoplaced)
