File: OBJEX-DoorSensor_v1.2/OBJEX-DoorSensor_v1.2.kicad_sch (KiCad schematic)
At the start: 5 parts

Commit message: Start PCB design
Parts:
- added U1: 5204, BatteryTerminal:5204, symbol BatteryTerminal:5204
- added U10: 5226, BatteryTerminal:5226, symbol BatteryTerminal:5226
Connections:
- net GND: now also U1.1 (-)
- net at D5.2 (A), JP1.1 (A), TP1.1: now also U10.1 (+)
Other:
- note added: "5204"
- note added: "5226"
- note removed: "5203"
- note removed: "5225"
- moved on the sheet: TP1, TP2
Changed lines of the file:
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@@
     (comment 2 "Designer: Salvatore Raccardi")
   )
+  (junction (at 54.61 85.09) (diameter 0) (color 0 0 0 0)
+  )
+  (junction (at 54.61 72.39) (diameter 0) (color 0 0 0 0)
+  )
   (junction (at 71.12 72.39) (diameter 0) (color 0 0 0 0)
-  )
-  (junction (at 55.88 72.39) (diameter 0) (color 0 0 0 0)
   )
   (no_connect (at 200.66 118.745))
@@
     (stroke (width 0) (type default))
   )
-  (polyline (pts (xy 43.18 62.23) (xy 43.18 96.52))
+  (wire (pts (xy 45.72 85.09) (xy 54.61 85.09))
+    (stroke (width 0) (type default))
+  )
+  (polyline (pts (xy 35.56 62.23) (xy 35.56 96.52))
     (stroke (width 0) (type dash_dot))
   )
@@
     (stroke (width 0) (type default))
   )
-  (wire (pts (xy 55.88 77.47) (xy 58.42 77.47))
-    (stroke (width 0) (type default))
-  )
-  (polyline (pts (xy 43.18 96.52) (xy 78.74 96.52))
+  (wire (pts (xy 54.61 77.47) (xy 58.42 77.47))
+    (stroke (width 0) (type default))
+  )
+  (polyline (pts (xy 35.56 96.52) (xy 78.74 96.52))
     (stroke (width 0) (type dash_dot))
   )
+  (wire (pts (xy 45.72 72.39) (xy 54.61 72.39))
+    (stroke (width 0) (type default))
+  )
+  (wire (pts (xy 54.61 71.12) (xy 54.61 72.39))
+    (stroke (width 0) (type default))
+  )
   (wire (pts (xy 71.12 85.09) (xy 71.12 87.63))
     (stroke (width 0) (type default))
@@
     (stroke (width 0) (type default))
   )
-  (polyline (pts (xy 77.47 62.23) (xy 43.18 62.23))
+  (polyline (pts (xy 77.47 62.23) (xy 35.56 62.23))
     (stroke (width 0) (type dash_dot))
   )
-  (wire (pts (xy 55.88 72.39) (xy 55.88 77.47))
-    (stroke (width 0) (type default))
-  )
-  (wire (pts (xy 55.88 72.39) (xy 58.42 72.39))
-    (stroke (width 0) (type default))
-  )
-  (wire (pts (xy 54.61 72.39) (xy 55.88 72.39))
+  (wire (pts (xy 54.61 72.39) (xy 58.42 72.39))
+    (stroke (width 0) (type default))
+  )
+  (wire (pts (xy 54.61 77.47) (xy 54.61 72.39))
     (stroke (width 0) (type default))
   )
@@
     (stroke (width 0) (type default))
   )
-  (rectangle (start 27.94 69.85) (end 33.655 91.44)
+  (rectangle (start 17.78 69.85) (end 23.495 91.44)
     (stroke (width 0) (type default))
     (fill (type none))
@@
     (fill (type none))
   )
-  (rectangle (start 33.655 69.85) (end 39.37 91.44)
+  (rectangle (start 23.495 69.85) (end 29.21 91.44)
     (stroke (width 0) (type default))
     (fill (type none))
@@
     (effects (font (size 1.2 1.2)) (justify left bottom))
   )
-  (text "5225" (at 37.465 68.58 90)
+  (text "5226\n" (at 27.305 68.58 90)
     (effects (font (size 1.27 1.27) bold italic) (justify left bottom))
   )
-  (text "+" (at 36.83 73.66 90)
+  (text "+" (at 26.67 73.66 90)
     (effects (font (size 1.27 1.27)) (justify left bottom))
   )
-  (text "-\n" (at 31.75 73.66 90)
+  (text "-\n" (at 21.59 73.66 90)
     (effects (font (size 1.27 1.27)) (justify left bottom))
   )
@@
     (effects (font (size 4 4) (thickness 0.6) bold) (justify left bottom))
   )
-  (text "+" (at 31.75 90.17 90)
+  (text "+" (at 21.59 90.17 90)
     (effects (font (size 1.27 1.27)) (justify left bottom))
   )
-  (text "--5213--\n" (at 39.37 93.98 0)
+  (text "--5213--\n" (at 29.21 93.98 0)
     (effects (font (size 1.27 1.27) (thickness 0.254) bold italic) (justify right bottom))
   )
-  (text "-\n" (at 36.83 90.17 90)
+  (text "-\n" (at 26.67 90.17 90)
     (effects (font (size 1.27 1.27)) (justify left bottom))
   )
-  (text "5203\n" (at 31.75 68.58 90)
+  (text "5204\n" (at 21.59 68.58 90)
     (effects (font (size 1.27 1.27) (thickness 0.254) bold italic) (justify left bottom))
   )
@@
     )
   )
-  (symbol (lib_id "Connector:TestPoint") (at 54.61 85.09 90) (unit 1)
+  (symbol (lib_id "Connector:TestPoint") (at 54.61 85.09 180) (unit 1)
     (in_bom yes) (on_board yes) (dnp no)
-    (property "Reference" "TP2" (at 53.975 83.82 90)
-      (effects (font (size 1.27 1.27)))
-    )
-    (property "Value" "GND" (at 48.26 85.09 90)
-      (effects (font (size 1.27 1.27)))
-    )
-    (property "Footprint" "TestPoint:TestPoint_Pad_1.5x1.5mm" (at 54.61 80.01 0)
-      (effects (font (size 1.27 1.27)) hide)
-    )
-    (property "Datasheet" "~" (at 54.61 80.01 0)
+    (property "Reference" "TP2" (at 52.07 86.36 0)
+      (effects (font (size 1.27 1.27)))
+    )
+    (property "Value" "GND" (at 54.61 91.44 90)
+      (effects (font (size 1.27 1.27)))
+    )
+    (property "Footprint" "TestPoint:TestPoint_Pad_1.5x1.5mm" (at 49.53 85.09 0)
+      (effects (font (size 1.27 1.27)) hide)
+    )
+    (property "Datasheet" "~" (at 49.53 85.09 0)
       (effects (font (size 1.27 1.27)) hide)
     )
@@
         (path "/dfd7f005-123d-49c6-a596-950b92e8aba7"
           (reference "TP2") (unit 1)
+        )
+      )
+    )
+  )
+  (symbol (lib_name "5226_1") (lib_id "BatteryTerminal:5226") (at 43.18 68.58 0) (unit 1)
+    (in_bom yes) (on_board yes) (dnp no)
+    (property "Reference" "U10" (at 42.5876 68.0136 0)
+      (effects (font (size 1.27 1.27)))
+    )
+    (property "Value" "5226" (at 43.18 69.85 0)
+      (effects (font (size 1.27 1.27)))
+    )
+    (property "Footprint" "BatteryTerminal:5226" (at 43.18 68.58 0)
+      (effects (font (size 1.27 1.27)) hide)
+    )
+    (property "Datasheet" "" (at 43.18 68.58 0)
+      (effects (font (size 1.27 1.27)) hide)
+    )
+    (pin "1")
+    (instances
+      (project "OBJEX-DoorSensor_v1.2"
+        (path "/dfd7f005-123d-49c6-a596-950b92e8aba7"
+          (reference "U10") (unit 1)
         )
       )
@@
     )
   )
+  (symbol (lib_id "BatteryTerminal:5204") (at 43.18 81.28 0) (unit 1)
+    (in_bom yes) (on_board yes) (dnp no)
+    (property "Reference" "U1" (at 41.91 80.01 0)
+      (effects (font (size 1.27 1.27)))
+    )
+    (property "Value" "5204" (at 43.18 82.55 0)
+      (effects (font (size 1.27 1.27)))
+    )
+    (property "Footprint" "BatteryTerminal:5204" (at 43.18 81.28 0)
+      (effects (font (size 1.27 1.27)) hide)
+    )
+    (property "Datasheet" "" (at 43.18 81.28 0)
+      (effects (font (size 1.27 1.27)) hide)
+    )
+    (pin "1")
+    (instances
+      (project "OBJEX-DoorSensor_v1.2"
+        (path "/dfd7f005-123d-49c6-a596-950b92e8aba7"
+          (reference "U1") (unit 1)
+        )
+      )
+    )
+  )
   (symbol (lib_id "power:GND") (at 168.148 122.8852 0) (unit 1)
     (in_bom yes) (on_board yes) (dnp no)
@@
     )
   )
-  (symbol (lib_id "Connector:TestPoint") (at 54.61 72.39 90) (unit 1)
+  (symbol (lib_id "Connector:TestPoint") (at 54.61 71.12 0) (unit 1)
     (in_bom yes) (on_board yes) (dnp no)
-    (property "Reference" "TP1" (at 53.975 71.12 90)
-      (effects (font (size 1.27 1.27)))
-    )
-    (property "Value" "BATT" (at 48.26 72.39 90)
-      (effects (font (size 1.27 1.27)))
-    )
-    (property "Footprint" "TestPoint:TestPoint_Pad_1.5x1.5mm" (at 54.61 67.31 0)
-      (effects (font (size 1.27 1.27)) hide)
-    )
-    (property "Datasheet" "~" (at 54.61 67.31 0)
-      (effects (font (size 1.27 1.27)) hide)
-    )
+    (property "Reference" "TP1" (at 52.07 69.85 0)
+      (effects (font (size 1.27 1.27)))
+    )
+    (property "Value" "BATT" (at 54.61 64.77 90)
+      (effects (font (size 1.27 1.27)))
+    )
+    (property "Footprint" "TestPoint:TestPoint_Pad_1.5x1.5mm" (at 59.69 71.12 0)
+      (effects (font (size 1.27 1.27)) hide)
+    )
+    (property "Datasheet" "~" (at 59.69 71.12 0)
+      (effects (font (size 1.27 1.27)) hide)
+    )

Commit message: last review
Changed lines of the file:
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@@
     (stroke (width 0) (type default))
   )
-  (polyline (pts (xy 35.56 62.23) (xy 35.56 96.52))
+  (polyline (pts (xy 35.56 62.23) (xy 35.56 95.25))
     (stroke (width 0) (type dash_dot))
   )
@@
     (stroke (width 0) (type default))
   )
-  (polyline (pts (xy 35.56 96.52) (xy 78.74 96.52))
+  (polyline (pts (xy 35.56 95.25) (xy 78.74 95.25))
     (stroke (width 0) (type dash_dot))
   )
@@
     (stroke (width 0) (type default))
   )
-  (rectangle (start 17.78 69.85) (end 23.495 91.44)
+  (rectangle (start 20.32 68.58) (end 26.035 90.17)
     (stroke (width 0) (type default))
     (fill (type none))
@@
     (fill (type none))
   )
-  (rectangle (start 23.495 69.85) (end 29.21 91.44)
+  (rectangle (start 26.035 68.58) (end 31.75 90.17)
     (stroke (width 0) (type default))
     (fill (type none))
@@
     (effects (font (size 1.2 1.2)) (justify left bottom))
   )
-  (text "5226\n" (at 27.305 68.58 90)
+  (text "5226\n" (at 29.845 67.31 90)
     (effects (font (size 1.27 1.27) bold italic) (justify left bottom))
   )
-  (text "+" (at 26.67 73.66 90)
+  (text "+" (at 29.21 72.39 90)
     (effects (font (size 1.27 1.27)) (justify left bottom))
   )
-  (text "-\n" (at 21.59 73.66 90)
+  (text "-\n" (at 24.13 72.39 90)
     (effects (font (size 1.27 1.27)) (justify left bottom))
   )
-  (text "Terminal\nBattery x2 AAA" (at 43.18 60.96 0)
+  (text "Terminal\nBattery x2 AAA" (at 43.18 59.69 0)
     (effects (font (size 2 2) (thickness 0.254) bold) (justify left bottom))
   )
@@
     (effects (font (size 4 4) (thickness 0.6) bold) (justify left bottom))
   )
-  (text "+" (at 21.59 90.17 90)
+  (text "+" (at 24.13 88.9 90)
     (effects (font (size 1.27 1.27)) (justify left bottom))
   )
-  (text "--5213--\n" (at 29.21 93.98 0)
+  (text "--5213--\n" (at 31.75 92.71 0)
     (effects (font (size 1.27 1.27) (thickness 0.254) bold italic) (justify right bottom))
   )
-  (text "-\n" (at 26.67 90.17 90)
+  (text "-\n" (at 29.21 88.9 90)
     (effects (font (size 1.27 1.27)) (justify left bottom))
   )
-  (text "5204\n" (at 21.59 68.58 90)
+  (text "5204\n" (at 24.13 67.31 90)
     (effects (font (size 1.27 1.27) (thickness 0.254) bold italic) (justify left bottom))
   )

Commit message: update
Changed lines of the file:
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@@
     )
-  )
-  (text "Copyright CERN 2020.\nThis source describes Open Hardware and is licensed under the CERN-OHLW v2\nYou may redistribute and modify this documentation and make products\nusing it under the terms of the CERN-OHL-W v2 (https:/cern.ch/cern-ohl).\nThis documentation is distributed WITHOUT ANY EXPRESS OR IMPLIED\nWARRANTY, INCLUDING OF MERCHANTABILITY, SATISFACTORY QUALITY\nAND FITNESS FOR A PARTICULAR PURPOSE. Please see the CERN-OHL-W v2\nfor applicable conditions.\nSource location: https://www.ohwr.org/project/wr-switch-hw\nAs per CERN-OHL-W v2 section 4.1, should You produce hardware based on\nthese sources, You must maintain the Source Location visible on the\nexternal case of the White Rabbit switch or other product you make using\nthis documentation."
-    (at 13.6652 194.9196 0)
-    (effects (font (size 1.2 1.2)) (justify left bottom))
   )
   (text "5226\n" (at 29.845 67.31 90)
@@
     (effects (font (size 1.27 1.27)) (justify left bottom))
   )
-  (text "Terminal\nBattery x2 AAA" (at 43.18 59.69 0)
+  (text "Copyright CERN 2020.\nThis source describes Open Hardware and is licensed under the CERN-OHLW v2\nYou may redistribute and modify this documentation and make products\nusing it under the terms of the CERN-OHL-W v2 (https:/cern.ch/cern-ohl).\nThis documentation is distributed WITHOUT ANY EXPRESS OR IMPLIED\nWARRANTY, INCLUDING OF MERCHANTABILITY, SATISFACTORY QUALITY\nAND FITNESS FOR A PARTICULAR PURPOSE. Please see the CERN-OHL-W v2\nfor applicable conditions.\nSource location: https://www.ohwr.org/project/wr-switch-hw\nAs per CERN-OHL-W v2 section 4.1, should You produce hardware based on\nthese sources, You must maintain the Source Location visible on the\nexternal case of the White Rabbit switch or other product you make using\nthis documentation."
+    (at 15.24 195.58 0)
+    (effects (font (size 2 2)) (justify left bottom))
+  )
+  (text "Terminal\nBattery x2 AAA" (at 35.56 59.69 0)
     (effects (font (size 2 2) (thickness 0.254) bold) (justify left bottom))
   )
