File: OBJEX-DoorSensor_v1.2/OBJEX-DoorSensor_v1.2.kicad_sch (KiCad schematic)
At the start: 7 parts, among them U1 5204, U10 5226

Commit message: bug fix
Other:
- note added: "USE 1N4148WS ONLY VBATT >= 3.7V"
Changed lines of the file:
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@@
+    (effects (font (size 1.27 1.27)) (justify left bottom))
+  )
+  (text "USE 1N4148WS ONLY VBATT >= 3.7V" (at 38.5826 98.7298 0)
     (effects (font (size 1.27 1.27)) (justify left bottom))
   )
