File: OBJEX-DoorSensor_v1.2/PowerLatch.kicad_sch (KiCad schematic)
At the start: 27 parts, among them Q1 BC857B_RF, Q2 NTNUS3171PZT5G, Q3 2N7002KQBZ, Q6 DMG3415UFY4Q-7, U3 S-5701BC11B-L3T2U5, U4 SN74LVC1G86DBVR, U5 SN74LVC1G86DBVR

Commit message: update
Parts:
- R9: value 1M -> 10K
Changed lines of the file:
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@@
       (effects (font (size 1.27 1.27)) (justify left))
     )
-    (property "Value" "1M" (at 105.41 104.775 0)
+    (property "Value" "10K" (at 105.41 104.775 0)
       (effects (font (size 1.27 1.27)) (justify left))
     )

Commit message: update
Parts:
- R10: value 1M -> 10K
- R6, R7: value 100M -> 1M
Changed lines of the file:
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@@
   (symbol (lib_id "Device:R") (at 45.72 87.63 0) (unit 1)
     (in_bom yes) (on_board yes) (dnp no) (fields_autoplaced)
-    (property "Reference" "R7" (at 48.0822 86.995 0)
-      (effects (font (size 1.27 1.27)) (justify left))
-    )
-    (property "Value" "100M" (at 48.0822 89.535 0)
+    (property "Reference" "R7" (at 48.26 86.995 0)
+      (effects (font (size 1.27 1.27)) (justify left))
+    )
+    (property "Value" "1M" (at 48.26 89.535 0)
       (effects (font (size 1.27 1.27)) (justify left))
     )
@@
       (effects (font (size 1.27 1.27)) (justify left))
     )
-    (property "Value" "1M" (at 105.41 117.475 0)
+    (property "Value" "10K" (at 105.41 117.475 0)
       (effects (font (size 1.27 1.27)) (justify left))
     )
@@
   (symbol (lib_id "Device:R") (at 45.72 77.47 0) (unit 1)
     (in_bom yes) (on_board yes) (dnp no) (fields_autoplaced)
-    (property "Reference" "R6" (at 48.0822 76.835 0)
-      (effects (font (size 1.27 1.27)) (justify left))
-    )
-    (property "Value" "100M" (at 48.0822 79.375 0)
-      (effects (font (size 1.27 1.27)) (justify left))
-    )
+    (property "Reference" "R6" (at 48.26 76.835 0)
+      (effects (font (size 1.27 1.27)) (justify left))
+    )
+    (property "Value" "1M" (at 48.26 79.375 0)
+      (effects (font (size 1.27 1.27)) (justify left))
+    )
