File: OBJEX-DoorSensor_v1.2/esp32c3.kicad_sch (KiCad schematic)
At the start: 10 parts, among them U1 ESP32-C3-MINI-1-N4, Y1 Crystal

Commit message: SCH complate
Parts:
- added D1: RED, LED_SMD:LED_0603_1608Metric, symbol Device:LED
- added D2: GREEN, LED_SMD:LED_0603_1608Metric, symbol Device:LED
- added D3: BLUE, LED_SMD:LED_0603_1608Metric, symbol Device:LED
- added R20, R21, R3: 1K, Resistor_SMD:R_0402_1005Metric, symbol Device:R
- added TP3: VBUS, TestPoint:TestPoint_Pad_D1.5mm, symbol Connector:TestPoint
- added TP4: TX, TestPoint:TestPoint_Pad_D1.5mm, symbol Connector:TestPoint
- added TP5: RX, TestPoint:TestPoint_Pad_D1.5mm, symbol Connector:TestPoint
- added TP6: RTS, TestPoint:TestPoint_Pad_D1.5mm, symbol Connector:TestPoint
- added TP7: DTR, TestPoint:TestPoint_Pad_D1.5mm, symbol Connector:TestPoint
- added TP8: GND, TestPoint:TestPoint_Pad_D1.5mm, symbol Connector:TestPoint
Connections:
- net GPIO2 is gone; now on net SDA: R1.1, U1.5 (IO2)
- net GPIO8 is gone; now on net SCL: R2.1, U1.22 (IO8)
- net +3V3: now also TP3.1
- net AUTO_TURN_OFF: now also U1.21 (IO7)
- net EN: now also TP6.1
- net GND: now also D1.1 (K), D2.1 (K), D3.1 (K), TP8.1
- net IN_STATUS: now also U1.18 (IO4)
- net RX/GPIO20: now also TP5.1
- net TX/GPIO21: now also TP4.1
- net D+: no longer names the net of U1.27 (IO19)
- net D-: no longer names the net of U1.26 (IO18)
- net GPIO10 renamed LED_GREEN
- net LED_GREEN: now also R20.2
- net GPIO5 renamed LED_BLUE
- net LED_BLUE: now also R21.2
- net GPIO6 renamed LED_RED
- net LED_RED: now also R3.2
- net GPIO9/DTR renamed DTR/GPIO9
- net DTR/GPIO9: now also TP7.1
- new net: D2.2 (A), R20.1
- new net: D1.2 (A), R3.1
- new net: D3.2 (A), R21.1
- no-connect marks 0 -> 2
Other:
- note added: "ESP32 TEST POINTs"
- moved on the sheet: C4, C5, Y1

Commit message: update
Parts:
- added D1: SP0503BAHT, Package_TO_SOT_SMD:SOT-143, symbol Power_Protection:SP0503BAHT
Connections:
- net +3V3: now also D1.3 (K)
- net GND: now also D1.1 (A)
- new net +BATT: D1.2 (K)
- no-connect marks 2 -> 3
Other:
- moved on the sheet: C1, C2, C3, C4, C5, R3, Y1

Commit message: Ready for components placing
Parts:
- U1: footprint XCVR_ESP32-C3-MINI-1-N4 -> lib:XCVR_ESP32-C3-MINI-1-N4
Changed lines of the file:
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@@
       (effects (font (size 1.27 1.27)))
     )
-    (property "Footprint" "XCVR_ESP32-C3-MINI-1-N4" (at 153.67 96.52 0)
+    (property "Footprint" "lib:XCVR_ESP32-C3-MINI-1-N4" (at 153.67 96.52 0)
       (effects (font (size 1.27 1.27)) (justify bottom) hide)
     )

Commit message: update
Parts:
- removed D1: SP0503BAHT, Package_TO_SOT_SMD:SOT-143, symbol Power_Protection:SP0503BAHT
Connections:
- no-connect marks 3 -> 2
Changed lines of the file:
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@@
   (no_connect (at 171.45 99.06))
   (no_connect (at 171.45 101.6))
-  (no_connect (at 81.28 156.21))
   (wire (pts (xy 125.73 96.52) (xy 135.89 96.52))
     (stroke (width 0) (type default))
   )
-  (wire (pts (xy 78.74 152.4) (xy 78.74 156.21))
-    (stroke (width 0) (type default))
-  )
   (wire (pts (xy 173.5328 114.3) (xy 173.5328 115.824))
     (stroke (width 0) (type default))
@@
     (stroke (width 0) (type default))
   )
-  (wire (pts (xy 74.93 153.67) (xy 76.2 153.67))
-    (stroke (width 0) (type default))
-  )
   (wire (pts (xy 218.44 105.41) (xy 218.44 114.3))
     (stroke (width 0) (type default))
   )
-  (wire (pts (xy 76.2 153.67) (xy 76.2 156.21))
-    (stroke (width 0) (type default))
-  )
   (wire (pts (xy 241.3 114.3) (xy 251.46 114.3))
     (stroke (width 0) (type default))
   )
   (wire (pts (xy 44.323 64.389) (xy 55.88 64.389))
-    (stroke (width 0) (type default))
-  )
-  (wire (pts (xy 78.74 166.37) (xy 78.74 168.91))
     (stroke (width 0) (type default))
   )
@@
     )
   )
-  (symbol (lib_name "+3V3_1") (lib_id "power:+3V3") (at 78.74 152.4 0) (unit 1)
-    (in_bom yes) (on_board yes) (dnp no) (fields_autoplaced)
-    (property "Reference" "#PWR051" (at 78.74 156.21 0)
-      (effects (font (size 1.27 1.27)) hide)
-    )
-    (property "Value" "+3V3" (at 78.74 148.59 0)
-      (effects (font (size 1.27 1.27)))
-    )
-    (property "Footprint" "" (at 78.74 152.4 0)
-      (effects (font (size 1.27 1.27)) hide)
-    )
-    (property "Datasheet" "" (at 78.74 152.4 0)
-      (effects (font (size 1.27 1.27)) hide)
-    )
-    (pin "1")
-    (instances
-      (project "OBJEX-DoorSensor_v1.2"
-        (path "/dfd7f005-123d-49c6-a596-950b92e8aba7/49ed0aa1-c89e-4756-9039-f42ff518440c"
-          (reference "#PWR051") (unit 1)
-        )
-      )
-    )
-  )
   (symbol (lib_id "Device:Crystal") (at 64.77 110.49 270) (unit 1)
     (in_bom yes) (on_board yes) (dnp no)
@@
     )
   )
-  (symbol (lib_id "Power_Protection:SP0503BAHT") (at 78.74 161.29 0) (unit 1)
-    (in_bom yes) (on_board yes) (dnp no)
-    (property "Reference" "D1" (at 83.947 160.1216 0)
-      (effects (font (size 1.27 1.27)) (justify left))
-    )
-    (property "Value" "SP0503BAHT" (at 83.947 162.433 0)
-      (effects (font (size 1.27 1.27)) (justify left))
-    )
-    (property "Footprint" "Package_TO_SOT_SMD:SOT-143" (at 84.455 162.56 0)
-      (effects (font (size 1.27 1.27)) (justify left) hide)
-    )
-    (property "Datasheet" "http://www.littelfuse.com/~/media/files/littelfuse/technical%20resources/documents/data%20sheets/sp05xxba.pdf" (at 81.915 158.115 0)
-      (effects (font (size 1.27 1.27)) hide)
-    )
-    (pin "1")
-    (pin "2")
-    (pin "3")
-    (pin "4")
-    (instances
-      (project "MainModule_v1.0"
-        (path "/234494ab-78d7-47dd-837d-036c186230fb"
-          (reference "D1") (unit 1)
-        )
-      )
-      (project "OBJEX-DoorSensor_v1.2"
-        (path "/dfd7f005-123d-49c6-a596-950b92e8aba7/49ed0aa1-c89e-4756-9039-f42ff518440c"
-          (reference "D4") (unit 1)
-        )
-      )
-    )
-  )
   (symbol (lib_id "Device:C") (at 56.261 104.267 270) (unit 1)
     (in_bom yes) (on_board yes) (dnp no)
@@
     )
   )
-  (symbol (lib_id "power:+BATT") (at 74.93 153.67 90) (unit 1)
-    (in_bom yes) (on_board yes) (dnp no) (fields_autoplaced)
-    (property "Reference" "#PWR012" (at 78.74 153.67 0)
-      (effects (font (size 1.27 1.27)) hide)
-    )
-    (property "Value" "+BATT" (at 71.12 154.305 90)
-      (effects (font (size 1.27 1.27)) (justify left))
-    )
-    (property "Footprint" "" (at 74.93 153.67 0)
-      (effects (font (size 1.27 1.27)) hide)
-    )
-    (property "Datasheet" "" (at 74.93 153.67 0)
-      (effects (font (size 1.27 1.27)) hide)
-    )
-    (pin "1")
-    (instances
-      (project "OBJEX-DoorSensor_v1.2"
-        (path "/dfd7f005-123d-49c6-a596-950b92e8aba7"
-          (reference "#PWR012") (unit 1)
-        )
-        (path "/dfd7f005-123d-49c6-a596-950b92e8aba7/92732d3f-bc3d-4824-8d12-1356e1adb506"
-          (reference "#PWR012") (unit 1)
-        )
-        (path "/dfd7f005-123d-49c6-a596-950b92e8aba7/49ed0aa1-c89e-4756-9039-f42ff518440c"
-          (reference "#PWR050") (unit 1)
-        )
-      )
-    )
-  )
   (symbol (lib_id "Connector:TestPoint") (at 36.83 162.56 90) (unit 1)
     (in_bom yes) (on_board yes) (dnp no)
@@
         )
       )
-    )
-  )
-  (symbol (lib_id "power:GND") (at 78.74 168.91 0) (unit 1)
-    (in_bom yes) (on_board yes) (dnp no)
-    (property "Reference" "#PWR022" (at 78.74 175.26 0)
-      (effects (font (size 1.27 1.27)) hide)
-    )
-    (property "Value" "GND" (at 78.867 173.3042 0)
-      (effects (font (size 1.27 1.27)))
-    )
-    (property "Footprint" "" (at 78.74 168.91 0)
-      (effects (font (size 1.27 1.27)) hide)
-    )
-    (property "Datasheet" "" (at 78.74 168.91 0)
-      (effects (font (size 1.27 1.27)) hide)
-    )
-    (pin "1")
-    (instances
-      (project "MainModule_v1.0"
-        (path "/234494ab-78d7-47dd-837d-036c186230fb"
-          (reference "#PWR022") (unit 1)
-        )
-      )
-      (project "OBJEX-DoorSensor_v1.2"
-        (path "/dfd7f005-123d-49c6-a596-950b92e8aba7/49ed0aa1-c89e-4756-9039-f42ff518440c"
-          (reference "#PWR052") (unit 1)
-        )
-      )

Commit message: update
Other:
- note added: "Copyright CERN 2020. This source describes Open Hardware and is licensed under the CERN-OHLW v2 You may redistribute and modify this documentation and make products using it under the terms of the CERN-OHL-W v2 (https:/cern.ch/cern-ohl). This documentation is distributed WITHOUT ANY EXPRESS OR IMPLIED WARRANTY, INCLUDING OF MERCHANTABILITY, SATISFACTORY QUALITY AND FITNESS FOR A PARTICULAR PURPOS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"
- moved on the sheet: C1, C2, C3, C4, C5, R3, TP3, TP4, TP5, TP6, TP7, TP8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
