File: ESP32-C3 Version/OBJEX-DoorSensor_v1.2/OBJEX-DoorSensor_v1.2.kicad_sch (KiCad schematic)
At the start: 7 parts, among them U1 5204, U10 5226

Commit message: update
Other:
- removed sheet Power Latch - Rising & falling edge detector 
- sheet Microcontroller + WiFi-BLE ports: added none; removed AUTO_TURN_OFF, BATT_LVL, IN_STATUS
- moved on the sheet: D5, JP1, TP1, TP2, U1, U10
