File: ESP32-C3 Version/OBJEX-DoorSensor_v1.2/RT9080.kicad_sch (KiCad schematic)
At the start: 4 parts, among them U6 RT9080-33GJ5

Commit message: update
Parts:
- renumbered C12 to C6, C6 to C7, R15 to R4, U6 to U2
