File: ESP32-C3 Version/OBJEX-DoorSensor_v1.2/esp32c3.kicad_sch (KiCad schematic)
At the start: 22 parts, among them U1 ESP32-C3-MINI-1-N4, Y1 Crystal

Commit message: update
Parts:
- renumbered C3 to C1, C4 to C2, C5 to C3, C1 to C4, C2 to C5, R3 to R1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
Connections:
- net AUTO_TURN_OFF: no longer names the net of U7.21 (IO7)
- net BATT_LVL: no longer names the net of U7.6 (IO3)
- net IN_STATUS: no longer names the net of U7.18 (IO4)
- no-connect marks 2 -> 5
